File: BudgetCANFD_G0.kicad_sch (KiCad schematic)
At the start: 86 parts, among them IC1 STM32G0B1KET6, IC2 M74VHC1GT66DTT1G, IC3 TJA1021TK_20_C,118, IC4 TPS56428DDA, IC5 NCV7356D1R2G, IC6 M74VHC1GT66DTT1G, J1 USB_C_Receptacle_USB2.0, J2 DB9_Male_MountingHoles, J3 20021511-00014T4LF, J4 Conn_01x02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

Commit message: Update to v1.1
Add support for an external clock if needed in the future
Parts:
- added C19: 0.1uF, Capacitor_SMD:C_0402_1005Metric, symbol Device:C
- added R30, R31: 0R, Resistor_SMD:R_0402_1005Metric, symbol Device:R_US
- added X1: SG-210STF, Oscillator:Oscillator_SMD_SeikoEpson_SG210-4Pin_2.5x2.0mm, symbol Oscillator:SG-210STF
- D3: Digi-Key_PN 475-3754-1-ND -> 475-2512-1-ND; LCSC Part # C72043 -> C2286; Manufacturer_Part_Number LG Q396-PS-35 -> LS Q976-NR-1
- F2: Digi-Key_PN (none) -> 507-2074-1-ND; LCSC Part # (none) -> C269145; Manufacturer_Part_Number (none) -> 0ZCG0200AF2B
- IC1: footprint QFP80P900X900X160-32N -> Package_QFP:LQFP-32_7x7mm_P0.8mm; LCSC Part # (none) -> C3223248
- IC2, IC6: footprint SOT65P210X110-5N -> Package_TO_SOT_SMD:SOT-353_SC-70-5; Digi-Key_PN (none) -> 296-24277-1-ND; LCSC Part # (none) -> C2673183
- IC3: footprint SON65P300X300X100-9N-D -> Package_SON:HVSON-8-1EP_3x3mm_P0.65mm_EP1.6x2.4mm
- IC5: footprint SOIC127P600X172-8N -> Package_SO:SOIC-8_3.9x4.9mm_P1.27mm
- L1: Digi-Key_PN (none) -> 587-2371-1-ND
- R1: Manufacturer_Part_Number RC0603FR-0710KL -> RC0603FR-07100KL
- R14: Digi-Key_PN (none) -> 311-470KHRCT-ND; Manufacturer_Part_Number (none) -> RC0603FR-07470KL
- R19: Digi-Key_PN 311-1.00KHRCT-ND -> 311-4.7KGRCT-ND; LCSC Part # C21190 -> C23162; Manufacturer_Part_Number RC0603FR-071KL -> RC0603JR-074K7L
- R21: Digi-Key_PN 311-1.00KHRCT-ND -> P6.49KFCT-ND; LCSC Part # C21190 -> (none); Manufacturer_Part_Number RC0603FR-071KL -> (none)
- R22: Digi-Key_PN 311-1.00KHRCT-ND -> 311-1.00KFRCT-ND
- SW1: Digi-Key_PN (none) -> CKN10723CT-ND; LCSC Part # (none) -> C221665; Manufacturer_Part_Number (none) -> JS202011JCQN
- SW1: footprint (none) -> Button_Switch_SMD:SW_DPDT_CK_JS202011JCQN; Digi-Key_PN (none) -> CKN10723CT-ND; LCSC Part # (none) -> C221665; Manufacturer_Part_Number (none) -> JS202011JCQN
- U1: Digi-Key_PN (none) -> 505-LTC4412ES6#TRPBFCT-ND; LCSC Part # C514442 -> C521306; Manufacturer_Part_Number (none) -> LTC4412xS6
- U2: Digi-Key_PN (none) -> AP2112K-3.3TRG1DICT-ND; Manufacturer_Part_Number (none) -> AP2112K-3.3
Connections:
- net +3V3: now also C19.1, X1.4 (Vcc)
- net GND: now also C19.2, X1.2 (GND)
- net STM32_OSC_IN: now reaches IC1.2 (PC14-OSC32_IN)
- net STM32_OSC_IN: now also R31.1
- net STM32_OSC_EN: now reaches IC1.3 (PC15-OSC32_OUT)
- net STM32_OSC_EN: now also R30.2
- new net: R30.1, X1.1 (~{ST})
- new net: R31.2, X1.3 (OUT)
- no-connect marks 15 -> 13
Other:
- company: (none) -> http://budgetcan.io
- title: (none) -> Budgetcan STM32G0B1xx

Commit message: Update BOM
Update part numbers for LCSC parts
Parts:
- C19: LCSC Part # C41851 -> C1525
- C20, C9: LCSC Part # C12891 -> C90146
- C7: value 0.47uF -> 4.7nF; LCSC Part # C2167812 -> C53987
- CR1, CR2: LCSC Part # C2831530 -> C58901
- IC2, IC6: LCSC Part # C2673183 -> C2762292
- R30, R31: LCSC Part # C15402 -> C60490
- X1: LCSC Part # C387448 -> C717682
Changed lines of the file:
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@@
     (pin "2")
     (pin "3")
+    (pin "4")
+    (pin "5")
+    (pin "6")
   )
   (symbol (lib_id "power:+3V3") (at 114.3 104.14 90) (unit 1)
@@
       (effects (font (size 1.27 1.27)) hide)
     )
-    (property "LCSC Part #" "C387448" (id 5) (at 62.23 142.24 0)
+    (property "LCSC Part #" "C717682" (id 5) (at 62.23 142.24 0)
       (effects (font (size 1.27 1.27)) hide)
     )
@@
       (effects (font (size 1.27 1.27)) hide)
     )
-    (property "LCSC Part #" "C15402" (id 5) (at 44.45 142.24 0)
+    (property "LCSC Part #" "C60490" (id 5) (at 44.45 142.24 0)
       (effects (font (size 1.27 1.27)) hide)
     )
@@
       (effects (font (size 1.27 1.27)) hide)
     )
+    (pin "1")
+    (pin "2")
+    (pin "3")
     (pin "4")
     (pin "5")
@@
       (effects (font (size 1.27 1.27)) hide)
     )
-    (property "LCSC Part #" "C15402" (id 5) (at 76.2 142.24 0)
+    (property "LCSC Part #" "C60490" (id 5) (at 76.2 142.24 0)
       (effects (font (size 1.27 1.27)) hide)
     )
@@
       (effects (font (size 1.524 1.524)))
     )
-    (property "LCSC Part #" "C2831530" (id 4) (at 353.06 237.49 0)
+    (property "LCSC Part #" "C58901" (id 4) (at 353.06 237.49 0)
       (effects (font (size 1.27 1.27)) hide)
     )
@@
       (effects (font (size 1.27 1.27)) hide)
     )
-    (property "LCSC Part #" "C12891" (id 4) (at 184.15 327.66 0)
+    (property "LCSC Part #" "C90146" (id 4) (at 184.15 327.66 0)
       (effects (font (size 1.27 1.27)) hide)
     )
@@
       (effects (font (size 1.27 1.27)) hide)
     )
-    (property "LCSC Part #" "C41851" (id 5) (at 52.07 128.27 0)
+    (property "LCSC Part #" "C1525" (id 5) (at 52.07 128.27 0)
       (effects (font (size 1.27 1.27)) hide)
     )
@@
       (effects (font (size 1.27 1.27)) (justify left) hide)
     )
-    (property "LCSC Part #" "C2673183" (id 10) (at 318.77 141.605 0)
+    (property "LCSC Part #" "C2762292" (id 10) (at 318.77 141.605 0)
       (effects (font (size 1.27 1.27)) hide)
     )
@@
       (effects (font (size 1.524 1.524)))
     )
-    (property "LCSC Part #" "C2831530" (id 4) (at 548.64 80.645 0)
+    (property "LCSC Part #" "C58901" (id 4) (at 548.64 80.645 0)
       (effects (font (size 1.27 1.27)) hide)
     )
@@
       (effects (font (size 1.27 1.27)) (justify left) hide)
     )
-    (property "LCSC Part #" "C2673183" (id 10) (at 429.26 143.51 0)
+    (property "LCSC Part #" "C2762292" (id 10) (at 429.26 143.51 0)
       (effects (font (size 1.27 1.27)) hide)
     )
@@
       (effects (font (size 1.27 1.27)) hide)
     )
-    (property "LCSC Part #" "C12891" (id 4) (at 196.215 226.06 0)
+    (property "LCSC Part #" "C90146" (id 4) (at 196.215 226.06 0)
       (effects (font (size 1.27 1.27)) hide)
     )
@@
       (effects (font (size 1.27 1.27)) (justify left))
     )
-    (property "Value" "0.47uF" (id 1) (at 173.736 236.093 0)
+    (property "Value" "4.7nF" (id 1) (at 173.736 236.093 0)
       (effects (font (size 1.27 1.27)) (justify left))
     )
@@
       (effects (font (size 1.27 1.27)) hide)
     )
-    (property "LCSC Part #" "C2167812" (id 4) (at 170.815 234.95 0)
+    (property "LCSC Part #" "C53987" (id 4) (at 170.815 234.95 0)
       (effects (font (size 1.27 1.27)) hide)
     )
@@
     )
     (path "/ed6554bb-befe-4fe8-b363-b041981d6e14"
-      (reference "C7") (unit 1) (value "0.47uF") (footprint "Capacitor_SMD:C_0603_1608Metric")
+      (reference "C7") (unit 1) (value "4.7nF") (footprint "Capacitor_SMD:C_0603_1608Metric")
     )
     (path "/2a305225-6f76-49bc-af47-29251428d058"

Commit message: Add BOM and updated part numbers
Parts:
- J2: Digi-Key_PN (none) -> AE10968-ND
- U4, U5: Digi-Key_PN (none) -> 568-13277-1-ND
Changed lines of the file:
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@@
+      (effects (font (size 1.27 1.27)) hide)
+    )
+    (property "Digi-Key_PN" "568-13277-1-ND" (id 5) (at 292.1 86.36 0)
       (effects (font (size 1.27 1.27)) hide)
     )
@@
       (effects (font (size 1.27 1.27)) hide)
     )
+    (property "Digi-Key_PN" "AE10968-ND" (id 4) (at 485.14 287.02 0)
+      (effects (font (size 1.27 1.27)) hide)
+    )
     (pin "0")
     (pin "1")
@@
       (effects (font (size 1.27 1.27)) hide)
     )
+    (property "Digi-Key_PN" "568-13277-1-ND" (id 5) (at 402.59 88.265 0)
+      (effects (font (size 1.27 1.27)) hide)
+    )
